File: pwr-conn/KiCad/PowConnV1.sch (KiCad schematic (older format))
At the start: 5 parts, among them P1 8Pin_2x4_inline, P2 PAD, P3 PAD, P4 PAD, P5 PAD

Commit message: kicad files, ready for assembly
as processed for the mfg+assembly .zip
Other:
- moved on the sheet: P1, P2, P3, P4, P5
Changed lines of the file:
@@
 EELAYER 26 0
 EELAYER END
-$Descr A4 11693 8268
+$Descr A 11000 8500
 encoding utf-8
 Sheet 1 1
-Title "PowConn"
-Date "2018-12-04"
-Rev "V1"
+Title "G935F-PWR"
+Date "2019-05-03"
+Rev "V2"
 Comp "Roman Dasovic"
 Comment1 ""
@@
 Comment4 ""
 $EndDescr
-Text GLabel 2950 2475 2    35   Input ~ 0
+Text GLabel 4450 3700 2    35   Input ~ 0
 Dev+
 $Comp
 L __SimpleParts:GND #PWR0105
 U 1 1 5C06F23E
-P 3550 2600
-F 0 "#PWR0105" H 3525 2585 5   0001 C CNN
-F 1 "GND" H 3520 2595 5   0001 C CNN
-F 2 "" H 3550 2600 50  0000 C CNN
-F 3 "" H 3550 2600 50  0000 C CNN
-	1    3550 2600
+P 5425 3850
+F 0 "#PWR0105" H 5400 3835 5   0001 C CNN
+F 1 "GND" H 5395 3845 5   0001 C CNN
+F 2 "" H 5425 3850 50  0000 C CNN
+F 3 "" H 5425 3850 50  0000 C CNN
+	1    5425 3850
 	0    1    1    0
 $EndComp
@@
 L __Interfaces:8Pin_2x4_inline P1
 U 1 1 5C0703E6
-P 2625 2550
-F 0 "P1" H 2625 2711 10  0000 C CNN
-F 1 "8Pin_2x4_inline" H 2625 2688 5   0000 C CNN
-F 2 "Footprints:8pin_molex_s7BatteryConn_5050040810" H 2620 2545 2   0001 C CNN
-F 3 "" H 2620 2545 20  0000 C CNN
-F 4 "Molex" H 2625 2525 10  0001 C CNN "Manufacturer1"
-F 5 "5050040810" H 2625 2550 10  0001 C CNN "Manufacturer1PartNumber"
-	1    2625 2550
+P 4125 3775
+F 0 "P1" H 4125 3936 10  0000 C CNN
+F 1 "8Pin_2x4_inline" H 4125 3913 5   0000 C CNN
+F 2 "Footprints:8pin_molex_s7BatteryConn_5050040810" H 4120 3770 2   0001 C CNN
+F 3 "" H 4120 3770 20  0000 C CNN
+F 4 "Molex" H 4125 3750 10  0001 C CNN "Manufacturer1"
+F 5 "5050040810" H 4125 3775 10  0001 C CNN "Manufacturer1PartNumber"
+	1    4125 3775
 	1    0    0    -1
 $EndComp
-Text Notes 2325 2275 0    50   ~ 0
+Text Notes 3825 3500 0    50   ~ 0
 S7 Battery Connector
 Wire Wire Line
-	2475 2700 2475 2625
+	3975 3925 3975 3850
 Wire Wire Line
-	2475 2625 2550 2625
+	3975 3850 4050 3850
 Wire Wire Line
-	2475 2625 2475 2575
+	3975 3850 3975 3800
 Wire Wire Line
-	2475 2575 2550 2575
-Connection ~ 2475 2625
+	3975 3800 4050 3800
+Connection ~ 3975 3850
 Wire Wire Line
-	2950 2475 2850 2475
+	4450 3700 4350 3700
 Wire Wire Line
-	2700 2525 2850 2525
+	4200 3750 4350 3750
 Wire Wire Line
-	2850 2525 2850 2475
-Connection ~ 2850 2475
+	4350 3750 4350 3700
+Connection ~ 4350 3700
 Wire Wire Line
-	2850 2475 2700 2475
+	4350 3700 4200 3700
 $Comp
 L __SimpleParts:PAD P2
 U 1 1 5C070C8F
-P 3025 3000
-F 0 "P2" H 3063 3000 10  0000 L CNN
-F 1 "PAD" H 3025 3000 3   0001 C CNN
-F 2 "Footprints:NPTH_1.5mm" H 2925 2925 60  0001 C CNN
-F 3 "" H 3055 3000 60  0001 C CNN
-F 4 "MFG1" H 3025 2975 6   0001 C CNN "Manufacturer1"
-F 5 "MFG1PN" H 3025 3000 6   0001 C CNN "Manufacturer1PartNumber"
-	1    3025 3000
+P 4800 4350
+F 0 "P2" H 4838 4350 10  0000 L CNN
+F 1 "PAD" H 4800 4350 3   0001 C CNN
+F 2 "Footprints:NPTH_1.5mm" H 4700 4275 60  0001 C CNN
+F 3 "" H 4830 4350 60  0001 C CNN
+F 4 "MFG1" H 4800 4325 6   0001 C CNN "Manufacturer1"
+F 5 "MFG1PN" H 4800 4350 6   0001 C CNN "Manufacturer1PartNumber"
+	1    4800 4350
 	1    0    0    -1
 $EndComp
-Text Notes 2950 2950 0    50   ~ 0
+Text Notes 4725 4300 0    50   ~ 0
 Drill Holes
 $Comp
 L __SimpleParts:PAD P3
 U 1 1 5C07170F
-P 3175 3000
-F 0 "P3" H 3213 3000 10  0000 L CNN
-F 1 "PAD" H 3175 3000 3   0001 C CNN
-F 2 "Footprints:NPTH_1.5mm" H 3075 2925 60  0001 C CNN
-F 3 "" H 3205 3000 60  0001 C CNN
-F 4 "MFG1" H 3175 2975 6   0001 C CNN "Manufacturer1"
-F 5 "MFG1PN" H 3175 3000 6   0001 C CNN "Manufacturer1PartNumber"
-	1    3175 3000
+P 4950 4350
+F 0 "P3" H 4988 4350 10  0000 L CNN
+F 1 "PAD" H 4950 4350 3   0001 C CNN
+F 2 "Footprints:NPTH_1.5mm" H 4850 4275 60  0001 C CNN
+F 3 "" H 4980 4350 60  0001 C CNN
+F 4 "MFG1" H 4950 4325 6   0001 C CNN "Manufacturer1"
+F 5 "MFG1PN" H 4950 4350 6   0001 C CNN "Manufacturer1PartNumber"
+	1    4950 4350
 	1    0    0    -1
 $EndComp
@@
 L __SimpleParts:PAD P4
 U 1 1 5C071890
-P 3750 2450
-F 0 "P4" H 3788 2450 10  0000 L CNN
-F 1 "PAD" H 3750 2450 3   0001 C CNN
-F 2 "Footprints:PAD_2.1mm_circle" H 3650 2375 60  0001 C CNN
-F 3 "" H 3780 2450 60  0001 C CNN
-F 4 "MFG1" H 3750 2425 6   0001 C CNN "Manufacturer1"
-F 5 "MFG1PN" H 3750 2450 6   0001 C CNN "Manufacturer1PartNumber"
-	1    3750 2450
+P 5625 3700
+F 0 "P4" H 5663 3700 10  0000 L CNN
+F 1 "PAD" H 5625 3700 3   0001 C CNN
+F 2 "Footprints:PAD_2.1mm_circle" H 5525 3625 60  0001 C CNN
+F 3 "" H 5655 3700 60  0001 C CNN
+F 4 "MFG1" H 5625 3675 6   0001 C CNN "Manufacturer1"
+F 5 "MFG1PN" H 5625 3700 6   0001 C CNN "Manufacturer1PartNumber"
+	1    5625 3700
 	1    0    0    -1
 $EndComp
-Text Notes 3575 2400 0    40   ~ 0
+Text Notes 5325 3550 0    40   ~ 0
 Pad Receiver for\nMain Board Spring clip
 $Comp
 L __SimpleParts:PAD P5
 U 1 1 5C072272
-P 3750 2600
-F 0 "P5" H 3788 2600 10  0000 L CNN
-F 1 "PAD" H 3750 2600 3   0001 C CNN
-F 2 "Footprints:PAD_2.1mm_circle" H 3650 2525 60  0001 C CNN
-F 3 "" H 3780 2600 60  0001 C CNN
-F 4 "MFG1" H 3750 2575 6   0001 C CNN "Manufacturer1"
-F 5 "MFG1PN" H 3750 2600 6   0001 C CNN "Manufacturer1PartNumber"
-	1    3750 2600
+P 5625 3850
+F 0 "P5" H 5663 3850 10  0000 L CNN
+F 1 "PAD" H 5625 3850 3   0001 C CNN
+F 2 "Footprints:PAD_2.1mm_circle" H 5525 3775 60  0001 C CNN
+F 3 "" H 5655 3850 60  0001 C CNN
+F 4 "MFG1" H 5625 3825 6   0001 C CNN "Manufacturer1"
+F 5 "MFG1PN" H 5625 3850 6   0001 C CNN "Manufacturer1PartNumber"
+	1    5625 3850
 	1    0    0    -1
 $EndComp
-Text GLabel 3575 2450 0    35   Input ~ 0
+Text GLabel 5450 3700 0    35   Input ~ 0
 Dev+
 Wire Wire Line
-	3575 2450 3750 2450
+	5450 3700 5625 3700
 Wire Wire Line
-	3550 2600 3750 2600
+	5425 3850 5625 3850
 $Comp
 L __SimpleParts:GND #PWR?
 U 1 1 5C0724CB
-P 2475 2700
-F 0 "#PWR?" H 2450 2685 5   0001 C CNN
-F 1 "GND" H 2445 2695 5   0001 C CNN
-F 2 "" H 2475 2700 50  0000 C CNN
-F 3 "" H 2475 2700 50  0000 C CNN
-	1    2475 2700
+P 3975 3925
+F 0 "#PWR?" H 3950 3910 5   0001 C CNN
+F 1 "GND" H 3945 3920 5   0001 C CNN
+F 2 "" H 3975 3925 50  0000 C CNN
+F 3 "" H 3975 3925 50  0000 C CNN
+	1    3975 3925
 	1    0    0    -1
 $EndComp
