File: usb-conn/KiCad/USBxtendV1.kicad_pcb (KiCad board)
At the start: 2 copper layers, 22.5 x 6 mm, 2 parts, among them P1 Conn_USB_5+Shell, P2 Conn_Basic_10_pin

Commit message: Ready for production
KiCAD source files and PCB manufacturing and assembly outputs.
Other:
- board text added: "2019-05-03"
- board text added: "Assembly Instructions:"
- board text added: "Copper Layers: 2 Soldermask Layers: 2 Silkscreen Layers: 2 All Layers: Trace Width / Trace Spacing : 6/6 mil Outer Layers: 1 oz copper Inner Layers: .5 oz copper Minimum Via Annular Ring / Drill Diameter: 25mil / 12mil Dielectric: FR-4 Finished board thickness: 1.0mm +- 10%"
- board text added: "Direction of Unreeling"
- board text added: "FILE DESCRIPTIONS:"
- board text added: "Figure 1"
- board text added: "Front Face Orientation"
- board text added: "G935-USB"
- board text added: "Orientation 0 degrees"
- board text added: "Orientation 180 degrees"
- board text added: "Orientation 270 degrees"
- board text added: "Orientation 90 degrees"
- board text added: "PCB Manufacturing Requirements:"
- board text added: "Please ask for clarification if any instructions are unclear. Assembly Instructions: 1. The .POS file contains centroid X-Y data and orientation. Orientation is such that 0 degrees indicates placement as if the reel sprocket holes are NORTH of the component. Refer to Figure 1. Do not place any items labeled as DNU. 2. BOM.csv containts BOM, quantities, and part numbers. Please advise before makin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"
- board text added: "Reel"
- board text added: "Round Sprocket Holes"
- board text added: "~~~~~~~~~~~~~~~~~~~~~~~~~~~~~~~~~~~~~~~~~~~~~~~~~~~~~~~~~~~~~~~~~~~~~~~~~~~~~~~~~~~~~~~~~~~~~~~~~~~~~~~~~~~~~~~~~~~~~~~~~~~~~~~~~~~~~~~~~~~~~~~~~~~~~~~~~~~~~~~~~~~~~~ ~~~~~~~~~~~~~~~~~~~~~~~~~~~~~~~~~~~~~~~~~~~~~~~~~~~~~~~~~~~~~~~~~~~~~~~~~~~~~~~~~~~~~~~~~~~~~~~~~~~~~~~~~~~~~~~~~~~~~~~~~~~~~~~~~~~~~~~~~~~~~~~~~~~~~~~~~~~~~~~~~~~~~~ Manufacturing Gerber Files -- Files needed for PCB Manufacturing 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"
- board text removed: "18/12/06"
- board text removed: "USBXtendV1"
- board text removed: "USBxtend V1 sensorable.io"
